Commit message: Modified for the compatibility of ROS noetic

File: pxpincher_description/urdf/arm_hardware.xacro (robot description, xacro)
@@ -15,5 +15,5 @@
   <xacro:macro name="arm_mount" params="parent name color *origin">
     <joint name="${name}_joint" type="fixed">
-      <insert_block name="origin"/>
+      <xacro:insert_block name="origin"/>
       <parent link="${parent}"/>
       <child link="${name}_link"/>
@@ -49,5 +49,5 @@
   <xacro:macro name="finger_fixed" params="parent name color *origin">
     <joint name="${name}_joint" type="fixed">
-      <insert_block name="origin"/>
+      <xacro:insert_block name="origin"/>
       <parent link="${parent}"/>
       <child link="${name}_link"/>
@@ -83,5 +83,5 @@
   <xacro:macro name="dynamixel_AX12_fixed" params="parent name *origin">
     <joint name="${name}_joint" type="fixed">
-      <insert_block name="origin"/>
+      <xacro:insert_block name="origin"/>
       <parent link="${parent}"/>
       <child link="${name}_link"/>
@@ -117,5 +117,5 @@
   <xacro:macro name="bioloid_F10_fixed" params="parent name color *origin">
     <joint name="${name}_joint" type="fixed">
-      <insert_block name="origin"/>
+      <xacro:insert_block name="origin"/>
       <parent link="${parent}"/>
       <child link="${name}_link"/>
@@ -151,5 +151,5 @@
   <xacro:macro name="bioloid_F3_fixed" params="parent name color *origin">
     <joint name="${name}_joint" type="fixed">
-      <insert_block name="origin"/>
+      <xacro:insert_block name="origin"/>
       <parent link="${parent}"/>
       <child link="${name}_link"/>
@@ -185,5 +185,5 @@
   <xacro:macro name="bioloid_F3_revolute" params="parent name color llimit ulimit vlimit *origin">
     <joint name="${name}_joint" type="revolute">
-      <insert_block name="origin"/>
+      <xacro:insert_block name="origin"/>
       <axis xyz="0 0 -1"/>
       <limit effort="30" velocity="${vlimit}" lower="${llimit}" upper="${ulimit}"/>
@@ -222,5 +222,5 @@
   <xacro:macro name="bioloid_F2_revolute" params="parent name color llimit ulimit vlimit *origin">
     <joint name="${name}_joint" type="revolute">
-      <insert_block name="origin"/>
+      <xacro:insert_block name="origin"/>
       <axis xyz="0 1 0"/>
       <limit effort="30" velocity="${vlimit}" lower="${llimit}" upper="${ulimit}"/>
@@ -259,5 +259,5 @@
   <xacro:macro name="bioloid_F4_revolute" params="parent name color llimit ulimit vlimit *origin">
     <joint name="${name}_joint" type="revolute">
-      <insert_block name="origin"/>
+      <xacro:insert_block name="origin"/>
       <axis xyz="0 1 0"/>
       <limit effort="30" velocity="${vlimit}" lower="${llimit}" upper="${ulimit}"/>
@@ -296,5 +296,5 @@
   <xacro:macro name="gripper_finger_base" params="parent name color *origin">
     <joint name="${name}_joint" type="fixed">
-      <insert_block name="origin"/>
+      <xacro:insert_block name="origin"/>
       <parent link="${parent}"/>
       <child link="${name}_link"/>
@@ -338,5 +338,5 @@
       </inertial>
       <visual>
-        <insert_block name="origin"/>
+        <xacro:insert_block name="origin"/>
         <geometry>
           <mesh filename="package://pxpincher_description/meshes/pincher_finger.stl" scale=".01 .01 .01"/>
@@ -345,5 +345,5 @@
       </visual>
       <collision>
-        <insert_block name="origin"/>
+        <xacro:insert_block name="origin"/>
         <geometry>
           <box size="0.036 0.028 0.004"/>

File: pxpincher_description/urdf/pincher_arm.urdf.xacro (robot description, xacro)
@@ -1,44 +1,743 @@
-<?xml version="1.0"?>
+<?xml version="1.0" encoding="utf-8"?>
+<!-- =================================================================================== -->
+<!-- |    This document was autogenerated by xacro from pincher_arm.urdf.xacro         | -->
+<!-- |    EDITING THIS FILE BY HAND IS NOT RECOMMENDED                                 | -->
+<!-- =================================================================================== -->
 <!-- Describe URDF for PhantomX Pincher Arm -->
-<robot name="turtlebot_arm" xmlns:xacro="http://ros.org/wiki/xacro">
-    <!-- We can configure joints velocity limit and lower/upper limits
+<robot name="turtlebot_arm">
+  <!-- We can configure joints velocity limit and lower/upper limits
           to allow access to different operational areas, e.g. left handed vs. right handed robot -->
-   <xacro:property name="joints_vlimit" value="1.571"/>
-    <xacro:property name="pan_llimit" value="-1.17"/>
-    <xacro:property name="pan_ulimit" value="1.43"/>
-    <xacro:property name="shoulder_llimit" value="0"/>
-    <xacro:property name="shoulder_ulimit" value="2.00"/>
-    <xacro:property name="elbow_llimit" value="-2.17"/>
-    <xacro:property name="elbow_ulimit" value="0.01"/>
-    <xacro:property name="wrist_llimit" value="-1.25"/>
-    <xacro:property name="wrist_ulimit" value="1.68"/>
-    <!-- Included URDF Files -->
-     <!-- Pincher arm is same as Turtlebot -->
-    <xacro:include filename="$(find pxpincher_description)/urdf/turtlebot_arm.xacro"/>
-    <!-- As we don't have here a turtlebot base, add a base_link link as its location reference -->
-    <link name="base_link"/>
-    <!-- Turtlebot arm macro -->
-    <turtlebot_arm parent="base_link" color="Gray" gripper_color="Gray"   pincher_gripper="true" turtlebot_gripper="false">
-      <!-- Place the "floating" arm at the location it should be if mounted on a turtlebot,
-           as pick and place and other demos assume this location -->
-      <origin xyz="0.06 0 0.01"/>
-    </turtlebot_arm>
-<!-- Phantomx Arm mount/Controllerboard link-->
-<joint name="arm_mount_joint" type="fixed">
-   <!--origin xyz="-0.09 -0.06 -0.105" rpy="0 0 0"/-->
-   <origin xyz="0.04 0.0 -0.065" rpy="0 0 0"/>
-   <parent link="arm_base_link"/>
-   <child link="arm_mount_link"/>
-   <axis xyz="0 0 1"/>
- </joint>
-<link name="arm_mount_link">
- <visual>
-   <!--origin xyz="0.18 -0.01 0.05" rpy="0 0 7.85"/-->
-   <origin xyz="0.091 -0.1 0.0" rpy="0 0 1.57"/>
-   <geometry>
-     <mesh filename="package://pxpincher_description/meshes/arm_mount.stl" scale="0.01 0.01 0.01"/>
-    </geometry>
-   <material name="Gray"/>
-  </visual>
-</link>
+  <!-- Included URDF Files -->
+  <material name="White">
+    <color rgba="0.87 0.90 0.87 1.0"/>
+  </material>
+  <material name="Black">
+    <color rgba="0.08 0.08 0.08 1.0"/>
+  </material>
+  <material name="Gray">
+    <color rgba="0.2 0.2 0.21 1.0"/>
+  </material>
+  <material name="Green">
+    <color rgba="0.22 0.32 0.14 1.0"/>
+  </material>
+  <!-- As we don't have here a turtlebot base, add a base_link link as its location reference -->
+  <link name="base_link"/>
+  <link name="arm_base_link"/>
+  <joint name="arm_base_joint" type="fixed">
+    <origin xyz="0.06 0 0.01"/>
+    <parent link="base_link"/>
+    <child link="arm_base_link"/>
+  </joint>
+  <!-- fake gripper_link joint gives us a free servo!
+         this makes us 5DOF and saves you $44.90
+         that's a lot of coin! -->
+  <link name="gripper_link"/>
+  <joint name="gripper_link_joint" type="revolute">
+    <origin rpy="0 -1.57 0" xyz="0 0 0.112"/>
+    <parent link="arm_wrist_flex_link"/>
+    <child link="gripper_link"/>
+    <limit effort="30" lower="-3.14" upper="3.14" velocity="1"/>
+    <axis xyz="1 0 0"/>
+  </joint>
+  <joint name="arm_shoulder_pan_servo_joint" type="fixed">
+    <origin rpy="1.570795 0 1.570795" xyz="0 0 0"/>
+    <parent link="arm_base_link"/>
+    <child link="arm_shoulder_pan_servo_link"/>
+  </joint>
+  <link name="arm_shoulder_pan_servo_link">
+    <inertial>
+      <mass value="0.055"/>
+      <origin xyz="0 0 0"/>
+      <inertia ixx="0.000017012" ixy="0.0" ixz="0.0" iyy="0.000013258" iyz="0.0" izz="0.000009483"/>
+    </inertial>
+    <visual>
+      <origin rpy="0 0 0" xyz=" 0 0 0 "/>
+      <geometry>
+        <mesh filename="package://pxpincher_description/meshes/ax12_box.stl" scale="0.001 0.001 0.001"/>
+      </geometry>
+      <material name="Black"/>
+    </visual>
+    <collision>
+      <origin rpy="0 0 0" xyz="0.0 0.0 -0.01241"/>
+      <geometry>
+        <box size="0.025 0.038 0.04762"/>
+      </geometry>
+    </collision>
+  </link>
+  <gazebo reference="arm_shoulder_pan_servo_link">
+    <material>Gazebo/Black</material>
+    <selfCollide>true</selfCollide>
+    <gravity>true</gravity>
+  </gazebo>
+  <joint name="arm_shoulder_pan_joint" type="revolute">
+    <origin rpy="-1.570795 1.570795 3.14159" xyz="0 0.019 0"/>
+    <axis xyz="0 0 -1"/>
+    <limit effort="30" lower="-1.17" upper="1.43" velocity="1.571"/>
+    <dynamics friction="0.13"/>
+    <parent link="arm_shoulder_pan_servo_link"/>
+    <child link="arm_shoulder_pan_link"/>
+  </joint>
+  <link name="arm_shoulder_pan_link">
+    <inertial>
+      <mass value="0.008"/>
+      <origin xyz="0 0 0"/>
+      <inertia ixx="0.000001" ixy="0.0" ixz="0.0" iyy="0.000001" iyz="0.0" izz="0.000001"/>
+    </inertial>
+    <visual>
+      <origin rpy="0 0 0" xyz=" 0 0 0 "/>
+      <geometry>
+        <mesh filename="package://pxpincher_description/meshes/F3.stl" scale="0.001 0.001 0.001"/>
+      </geometry>
+      <material name="Gray"/>
+    </visual>
+    <collision>
+      <origin rpy="0 0 0" xyz="0.0 0.0 -0.0045"/>
+      <geometry>
+        <box size="0.025 0.038 0.009"/>
+      </geometry>
+    </collision>
+  </link>
+  <gazebo reference="arm_shoulder_pan_link">
+    <material>Gazebo/Gray</material>
+    <selfCollide>true</selfCollide>
+    <gravity>true</gravity>
+  </gazebo>
+  <joint name="arm_shoulder_lift_servo_joint" type="fixed">
+    <origin rpy="0 3.14159 0" xyz="0 0 -0.0415"/>
+    <parent link="arm_shoulder_pan_link"/>
+    <child link="arm_shoulder_lift_servo_link"/>
+  </joint>
+  <link name="arm_shoulder_lift_servo_link">
+    <inertial>
+      <mass value="0.055"/>
+      <origin xyz="0 0 0"/>
+      <inertia ixx="0.000017012" ixy="0.0" ixz="0.0" iyy="0.000013258" iyz="0.0" izz="0.000009483"/>
+    </inertial>
+    <visual>
+      <origin rpy="0 0 0" xyz=" 0 0 0 "/>
+      <geometry>
+        <mesh filename="package://pxpincher_description/meshes/ax12_box.stl" scale="0.001 0.001 0.001"/>
+      </geometry>
+      <material name="Black"/>
+    </visual>
+    <collision>
+      <origin rpy="0 0 0" xyz="0.0 0.0 -0.01241"/>
+      <geometry>
+        <box size="0.025 0.038 0.04762"/>
+      </geometry>
+    </collision>
+  </link>
+  <gazebo reference="arm_shoulder_lift_servo_link">
+    <material>Gazebo/Black</material>
+    <selfCollide>true</selfCollide>
+    <gravity>true</gravity>
+  </gazebo>
+  <joint name="arm_shoulder_lift_joint" type="revolute">
+    <origin rpy="0 0 0" xyz="0 0 0"/>
+    <axis xyz="0 1 0"/>
+    <limit effort="30" lower="0" upper="2.0" velocity="1.571"/>
+    <dynamics friction="0.13"/>
+    <parent link="arm_shoulder_lift_servo_link"/>
+    <child link="arm_shoulder_lift_link"/>
+  </joint>
+  <link name="arm_shoulder_lift_link">
+    <inertial>
+      <mass value="0.016"/>
+      <origin xyz="0 0 0"/>
+      <inertia ixx="0.000001" ixy="0.0" ixz="0.0" iyy="0.000001" iyz="0.0" izz="0.000001"/>
+    </inertial>
+    <visual>
+      <origin rpy="0 0 0" xyz=" 0 0 0 "/>
+      <geometry>
+        <mesh filename="package://pxpincher_description/meshes/F4.stl" scale="0.001 0.001 0.001"/>
+      </geometry>
+      <material name="Gray"/>
+    </visual>
+    <collision>
+      <origin rpy="0 0 0" xyz="0.0 0.0 0.0215"/>
+      <geometry>
+        <box size="0.028 0.0485 0.065"/>
+      </geometry>
+    </collision>
+  </link>
+  <gazebo reference="arm_shoulder_lift_link">
+    <material>Gazebo/Gray</material>
+    <selfCollide>true</selfCollide>
+    <gravity>true</gravity>
+  </gazebo>
+  <joint name="arm_shoulder_F10_0_joint" type="fixed">
+    <origin rpy="0 0 0" xyz="0 0 0.0545"/>
+    <parent link="arm_shoulder_lift_link"/>
+    <child link="arm_shoulder_F10_0_link"/>
+  </joint>
+  <link name="arm_shoulder_F10_0_link">
+    <inertial>
+      <mass value="0.004"/>
+      <origin xyz="0 0 0"/>
+      <inertia ixx="0.000001" ixy="0.0" ixz="0.0" iyy="0.000001" iyz="0.0" izz="0.000001"/>
+    </inertial>
+    <visual>
+      <origin rpy="0 0 0" xyz=" 0 0 0 "/>
+      <geometry>
+        <mesh filename="package://pxpincher_description/meshes/F10.stl" scale="0.001 0.001 0.001"/>
+      </geometry>
+      <material name="Gray"/>
+    </visual>
+    <collision>
+      <origin rpy="0 0 0" xyz="0.0 0.0 0.0"/>
+      <geometry>
+        <box size="0.025 0.038 0.004"/>
+      </geometry>
+    </collision>
+  </link>
+  <gazebo reference="arm_shoulder_F10_0_link">
+    <material>Gazebo/Gray</material>
+    <selfCollide>true</selfCollide>
+    <gravity>true</gravity>
+  </gazebo>
+  <joint name="arm_shoulder_F10_1_joint" type="fixed">
+    <origin rpy="0 0 0" xyz="0 0 0.004"/>
+    <parent link="arm_shoulder_F10_0_link"/>
+    <child link="arm_shoulder_F10_1_link"/>
+  </joint>
+  <link name="arm_shoulder_F10_1_link">
+    <inertial>
+      <mass value="0.004"/>
+      <origin xyz="0 0 0"/>
+      <inertia ixx="0.000001" ixy="0.0" ixz="0.0" iyy="0.000001" iyz="0.0" izz="0.000001"/>
+    </inertial>
+    <visual>
+      <origin rpy="0 0 0" xyz=" 0 0 0 "/>
+      <geometry>
+        <mesh filename="package://pxpincher_description/meshes/F10.stl" scale="0.001 0.001 0.001"/>
+      </geometry>
+      <material name="Gray"/>
+    </visual>
+    <collision>
+      <origin rpy="0 0 0" xyz="0.0 0.0 0.0"/>
+      <geometry>
+        <box size="0.025 0.038 0.004"/>
+      </geometry>
+    </collision>
+  </link>
+  <gazebo reference="arm_shoulder_F10_1_link">
+    <material>Gazebo/Gray</material>
+    <selfCollide>true</selfCollide>
+    <gravity>true</gravity>
+  </gazebo>
+  <joint name="arm_shoulder_F10_2_joint" type="fixed">
+    <origin rpy="0 0 0" xyz="0 0 0.004"/>
+    <parent link="arm_shoulder_F10_1_link"/>
+    <child link="arm_shoulder_F10_2_link"/>
+  </joint>
+  <link name="arm_shoulder_F10_2_link">
+    <inertial>
+      <mass value="0.004"/>
+      <origin xyz="0 0 0"/>
+      <inertia ixx="0.000001" ixy="0.0" ixz="0.0" iyy="0.000001" iyz="0.0" izz="0.000001"/>
+    </inertial>
+    <visual>
+      <origin rpy="0 0 0" xyz=" 0 0 0 "/>
+      <geometry>
+        <mesh filename="package://pxpincher_description/meshes/F10.stl" scale="0.001 0.001 0.001"/>
+      </geometry>
+      <material name="Gray"/>
+    </visual>
+    <collision>
+      <origin rpy="0 0 0" xyz="0.0 0.0 0.0"/>
+      <geometry>
+        <box size="0.025 0.038 0.004"/>
+      </geometry>
+    </collision>
+  </link>
+  <gazebo reference="arm_shoulder_F10_2_link">
+    <material>Gazebo/Gray</material>
+    <selfCollide>true</selfCollide>
+    <gravity>true</gravity>
+  </gazebo>
+  <joint name="arm_shoulder_F3_0_joint" type="fixed">
+    <origin rpy="0 3.14159 0" xyz="0 0 0.002"/>
+    <parent link="arm_shoulder_F10_2_link"/>
+    <child link="arm_shoulder_F3_0_link"/>
+  </joint>
+  <link name="arm_shoulder_F3_0_link">
+    <inertial>
+      <mass value="0.005"/>
+      <origin xyz="0 0 0"/>
+      <inertia ixx="0.000001" ixy="0.0" ixz="0.0" iyy="0.000001" iyz="0.0" izz="0.000001"/>
+    </inertial>
+    <visual>
+      <origin rpy="0 0 0" xyz=" 0 0 0 "/>
+      <geometry>
+        <mesh filename="package://pxpincher_description/meshes/F3.stl" scale="0.001 0.001 0.001"/>
+      </geometry>
+      <material name="Gray"/>
+    </visual>
+    <collision>
+      <origin rpy="0 0 0" xyz="0.0 0.0 -0.0045"/>
+      <geometry>
+        <box size="0.025 0.038 0.009"/>
+      </geometry>
+    </collision>
+  </link>
+  <gazebo reference="arm_shoulder_F3_0_link">
+    <material>Gazebo/Gray</material>
+    <selfCollide>true</selfCollide>
+    <gravity>true</gravity>
+  </gazebo>
+  <joint name="arm_elbow_flex_servo_joint" type="fixed">
+    <origin rpy="0 3.14159 0" xyz="0 0 -0.0415"/>
+    <parent link="arm_shoulder_F3_0_link"/>
+    <child link="arm_elbow_flex_servo_link"/>
+  </joint>
+  <link name="arm_elbow_flex_servo_link">
+    <inertial>
+      <mass value="0.055"/>
+      <origin xyz="0 0 0"/>
+      <inertia ixx="0.000017012" ixy="0.0" ixz="0.0" iyy="0.000013258" iyz="0.0" izz="0.000009483"/>
+    </inertial>
+    <visual>
+      <origin rpy="0 0 0" xyz=" 0 0 0 "/>
+      <geometry>
+        <mesh filename="package://pxpincher_description/meshes/ax12_box.stl" scale="0.001 0.001 0.001"/>
+      </geometry>
+      <material name="Black"/>
+    </visual>
+    <collision>
+      <origin rpy="0 0 0" xyz="0.0 0.0 -0.01241"/>
+      <geometry>
+        <box size="0.025 0.038 0.04762"/>
+      </geometry>
+    </collision>
+  </link>
+  <gazebo reference="arm_elbow_flex_servo_link">
+    <material>Gazebo/Black</material>
+    <selfCollide>true</selfCollide>
+    <gravity>true</gravity>
+  </gazebo>
+  <joint name="arm_elbow_flex_joint" type="revolute">
+    <origin rpy="0 0 0" xyz="0 0 0"/>
+    <axis xyz="0 1 0"/>
+    <limit effort="30" lower="-2.17" upper="0.01" velocity="1.571"/>
+    <dynamics friction="0.13"/>
+    <parent link="arm_elbow_flex_servo_link"/>
+    <child link="arm_elbow_flex_link"/>
+  </joint>
+  <link name="arm_elbow_flex_link">
+    <inertial>
+      <mass value="0.016"/>
+      <origin xyz="0 0 0"/>
+      <inertia ixx="0.000001" ixy="0.0" ixz="0.0" iyy="0.000001" iyz="0.0" izz="0.000001"/>
+    </inertial>
+    <visual>
+      <origin rpy="0 0 0" xyz=" 0 0 0 "/>
+      <geometry>
+        <mesh filename="package://pxpincher_description/meshes/F4.stl" scale="0.001 0.001 0.001"/>
+      </geometry>
+      <material name="Gray"/>
+    </visual>
+    <collision>
+      <origin rpy="0 0 0" xyz="0.0 0.0 0.0215"/>
+      <geometry>
+        <box size="0.028 0.0485 0.065"/>
+      </geometry>
+    </collision>
+  </link>
+  <gazebo reference="arm_elbow_flex_link">
+    <material>Gazebo/Gray</material>
+    <selfCollide>true</selfCollide>
+    <gravity>true</gravity>
+  </gazebo>
+  <joint name="arm_elbow_F10_0_joint" type="fixed">
+    <origin rpy="0 0 0" xyz="0 0 0.0545"/>
+    <parent link="arm_elbow_flex_link"/>
+    <child link="arm_elbow_F10_0_link"/>
+  </joint>
+  <link name="arm_elbow_F10_0_link">
+    <inertial>
+      <mass value="0.004"/>
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
File: pxpincher_description/urdf/turtlebot_arm.xacro (robot description, xacro)
@@ -18,5 +18,5 @@
     <link name="arm_base_link"/>
     <joint name="arm_base_joint" type="fixed">
-      <insert_block name="origin"/>
+      <xacro:insert_block name="origin"/>
       <parent link="${parent}"/>
       <child link="arm_base_link"/>
